File: ProjetoI/ProjetoI.kicad_pcb (KiCad board)
At the start: 2 copper layers, 41 x 35.5 mm, 17 parts, among them J1 PJ-002A, J3 USB_A, U1 MCP73833-xxx-UN

Commit message: final
Other:
- board text added: "Andrey Gregório Cassiano Lucas Souza de Oliveira Poliana Cruz Costa Victor Hugo Rodrigues"
Changed lines of the file:
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@@
 		(layer "Edge.Cuts")
+	)
+	(gr_text "Andrey Gregório Cassiano\nLucas Souza de Oliveira\nPoliana Cruz Costa\nVictor Hugo Rodrigues"
+		(at 116.5 110.5 90)
+		(layer "F.SilkS")
+		(effects
+			(font
+				(size 0.5 0.5)
+				(thickness 0.125)
+			)
+			(justify left bottom)
+		)
 	)
 	(segment
